Commit message: tentativa de melhoramento das funções de repulsão e ajuste de parâmetros

File: nav_bringup/urdf/diff_robot.urdf.xacro (robot description, xacro)
@@ -5,8 +5,8 @@
   <xacro:property name="base_width"  value="0.30"/>
   <xacro:property name="base_height" value="0.15"/>
-  <xacro:property name="base_mass"   value="5.0"/>
+  <xacro:property name="base_mass"   value="8.0"/>
   <xacro:property name="wheel_radius"    value="0.08"/>
   <xacro:property name="wheel_thickness" value="0.04"/>
-  <xacro:property name="wheel_mass"      value="0.5"/>
+  <xacro:property name="wheel_mass"      value="1.0"/>
   <xacro:property name="wheel_separation" value="0.34"/>
   <xacro:property name="caster_radius" value="0.04"/>
@@ -88,6 +88,7 @@
       <parent link="base_link"/>
       <child link="wheel_${prefix}"/>
-      <origin xyz="0 ${y_offset} ${-base_height/2}" rpy="0 0 0"/>
+      <origin xyz="0 ${y_offset} ${-base_height/2 + wheel_radius}" rpy="0 0 0"/>
       <axis xyz="0 1 0"/>
+      <dynamics damping="0.2" friction="0.1"/>
     </joint>
   </xacro:macro>
@@ -109,10 +110,10 @@
       </geometry>
     </collision>
-    <xacro:sphere_inertia m="0.1" r="${caster_radius}"/>
+    <xacro:sphere_inertia m="0.3" r="${caster_radius}"/>
   </link>
   <joint name="caster_joint" type="fixed">
     <parent link="base_link"/>
     <child link="caster"/>
-    <origin xyz="${-base_length/2 + caster_radius} 0 ${-base_height/2 - wheel_radius + caster_radius}"/>
+    <origin xyz="${-base_length/2 + caster_radius} 0 ${-base_height/2 + caster_radius}"/>
   </joint>
   <!-- ========== LASER ========== -->
@@ -140,10 +141,10 @@
   <!-- ========== GAZEBO: ATRITO DAS RODAS ========== -->
   <gazebo reference="wheel_left">
-    <mu1>1.0</mu1>
-    <mu2>1.0</mu2>
+    <mu1>0.6</mu1>
+    <mu2>0.6</mu2>
   </gazebo>
   <gazebo reference="wheel_right">
-    <mu1>1.0</mu1>
-    <mu2>1.0</mu2>
+    <mu1>0.6</mu1>
+    <mu2>0.6</mu2>
   </gazebo>
   <gazebo reference="caster">
